Commit message: Added rear lidar, implemented ros2_laser_scan_merger for two lidars.

File: src/wheeltec_robot_urdf/urdf/oplsim.urdf (robot description, URDF)
Before this commit: robot wheeltec_robot, 7 links, 6 joints
Links:
- added link rear_laser_link, mass 0.037; collision cylinder length=0.04 radius=0.035; visual mesh filename=package://wheeltec_robot_urdf/meshes/S100_diff_robot_meshes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
- link base_link: geometry collision box size=0.22 0.16 0.08; visual mesh filename=package://wheeltec_robot_urdf/meshes/S100_diff_robot_meshes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 scale=0.001 0.001 0.001
Joints:
- added joint rear_laser_joint: type fixed, parent base_link, child rear_laser_link, origin xyz=-0.12 0 0.18 rpy=0 0 3.141592653589793

Commit message: Update robot navigation and configuration

File: src/wheeltec_robot_urdf/urdf/oplsim.urdf (robot description, URDF)
Before this commit: robot wheeltec_robot, 8 links, 7 joints
Links:
- link base_link: geometry collision mesh filename=package://wheeltec_robot_urdf/meshes/S100_diff_robot_meshes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 scale=0.001 0.001 0.001; visual mesh filename=package://wheeltec_robot_urdf/meshes/S100_diff_robot_meshes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 scale=0.001 0.001 0.001
- link lf_wheel_link: geometry collision mesh filename=package://wheeltec_robot_urdf/meshes/S100_diff_robot_meshes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; visual mesh filename=package://wheeltec_robot_urdf/meshes/S100_diff_robot_meshes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
- link rf_wheel_link: geometry collision mesh filename=package://wheeltec_robot_urdf/meshes/S100_diff_robot_meshes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; visual mesh filename=package://wheeltec_robot_urdf/meshes/S100_diff_robot_meshes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
Joints:
- joint caster_left_joint: origin xyz=-0.12 0.08 0.018 rpy=0 0 0 -> xyz=-0.12 0.08 -0.01 rpy=0 0 0
- joint caster_right_joint: origin xyz=-0.12 -0.08 0.018 rpy=0 0 0 -> xyz=-0.12 -0.08 -0.01 rpy=0 0 0

Commit message: Fusing IMU

File: src/wheeltec_robot_urdf/urdf/oplsim.urdf (robot description, URDF)
Before this commit: robot wheeltec_robot, 20 links, 19 joints
Links:
- added link imu_link
- link Z_link: mass 0.037 -> 0.0001
- link arm_base: mass 0.162548567403693 -> 0.0001
- link link1: mass 0.0978679932242825 -> 0.0001
- link link2: mass 0.290888938633388 -> 0.0001
- link link3: mass 0.290847697793211 -> 0.0001
- link link4: mass 0.127087348341362 -> 0.0001
- link link5: mass 0.144711242639457 -> 0.0001
- link link6: mass 0.195187143240719 -> 0.0001
- link link7: mass 0.02648229234527 -> 0.0001
- link link8: mass 0.0264822021416248 -> 0.0001
Joints:
- added joint imu_joint: type fixed, parent rtab_cam_link, child imu_link, origin xyz=0 0 0 rpy=0 0 0

Commit message: Fixed camera optical joint

File: src/wheeltec_robot_urdf/urdf/oplsim.urdf (robot description, URDF)
Before this commit: robot wheeltec_robot, 21 links, 20 joints
Joints:
- joint rtab_cam_optical_joint: origin xyz=0.00615 0 0 rpy=0 0 0 -> xyz=0.00615 0 0 rpy=-1.57079632679 0 -1.57079632679
